Commit message: Created Gazebo_control

File: description/robot_core.xacro (robot description, xacro)
@@ -82,10 +82,10 @@
     </link>
 <!--========================================== right WHEEL JOINT ==========================================-->
-<joint name="wheel_right_joint" type="continuous">
-    <origin xyz="0 -0.158075 0.0255" rpy="-${pi/2} 0 0"/>
-    <parent link="base_link" />
-    <child link="wheel_right_link" />
-    <axis xyz="0 0 1 " />
-  </joint>
+    <joint name="wheel_right_joint" type="continuous">
+        <origin xyz="0 -0.158075 0.0255" rpy="-${pi/2} 0 0"/>
+        <parent link="base_link" />
+        <child link="wheel_right_link" />
+        <axis xyz="0 0 1 " />
+    </joint>
 <!--========================================== right WHEEL LINK ==========================================-->
     <link name="wheel_right_link">
@@ -108,56 +108,76 @@
             </geometry>
         </collision>
-  </link>
+    </link>
 <!--============================================ FRONT CASTOR WHEEL JOINT ============================================-->
     <joint name="caster_front_link_joint" type="fixed">
-    <origin xyz="0.2 0.0 -0.0145" rpy="0.0 0.0 0.0"/>
-    <parent link="base_link" />
-    <child link="caster_front_link" />
-    <axis xyz="0 0 0" />
+        <origin xyz="0.2 0.0 -0.0145" rpy="0.0 0.0 0.0"/>
+        <parent link="base_link" />
+        <child link="caster_front_link" />
+        <axis xyz="0 0 0" />
     </joint>
 <!--=============================================== FRONT CASTOR WHEEL LINK ===============================================-->
-<link name="caster_front_link">
-    <xacro:inertial_sphere mass="0.1" radius="0.025">
-        <origin xyz="0 0 0" rpy="0 0 0"/>
-    </xacro:inertial_sphere>
-    <visual>
-        <origin xyz="0 0 0" rpy="0 0 0" />
-        <geometry>
+    <link name="caster_front_link">
+        <xacro:inertial_sphere mass="0.1" radius="0.025">
+            <origin xyz="0 0 0" rpy="0 0 0"/>
+        </xacro:inertial_sphere>
+        <visual>
+            <origin xyz="0 0 0" rpy="0 0 0" />
+            <geometry>
+                <sphere radius="0.025" />
+            </geometry>
+            <material name="grey" />
+        </visual>
+        <collision>
+            <origin xyz="0 0 0" rpy="0 0 0" />
+            <geometry>
             <sphere radius="0.025" />
-        </geometry>
-        <material name="grey" />
-    </visual>
-    <collision>
-        <origin xyz="0 0 0" rpy="0 0 0" />
-        <geometry>
-          <sphere radius="0.025" />
-        </geometry>
-    </collision>
+            </geometry>
+        </collision>
+    </link>
 <!--============================================ REAR CASTOR WHEEL JOINT ============================================-->
     <joint name="caster_rear_link_joint" type="fixed">
-    <origin xyz="-0.2 0.0 -0.0145" rpy="0.0 0.0 0.0"/>
-    <parent link="base_link" />
-    <child link="caster_rear_link" />
-    <axis xyz="0 0 0" />
+        <origin xyz="-0.2 0.0 -0.0145" rpy="0.0 0.0 0.0"/>
+        <parent link="base_link" />
+        <child link="caster_rear_link" />
+        <axis xyz="0 0 0" />
     </joint>
-  <!--=============================================== REAR CASTOR WHEEL LINK ===============================================-->
-<link name="caster_rear_link">
-    <xacro:inertial_sphere mass="0.1" radius="0.025">
-        <origin xyz="0 0 0" rpy="0 0 0"/>
-    </xacro:inertial_sphere>
-    <visual>
-        <origin xyz="0 0 0" rpy="0 0 0" />
-        <geometry>
+<!--=============================================== REAR CASTOR WHEEL LINK ===============================================-->
+    <link name="caster_rear_link">
+        <xacro:inertial_sphere mass="0.1" radius="0.025">
+            <origin xyz="0 0 0" rpy="0 0 0"/>
+        </xacro:inertial_sphere>
+        <visual>
+            <origin xyz="0 0 0" rpy="0 0 0" />
+            <geometry>
+                <sphere radius="0.025" />
+            </geometry>
+            <material name="grey" />
+        </visual>
+        <collision>
+            <origin xyz="0 0 0" rpy="0 0 0" />
+            <geometry>
             <sphere radius="0.025" />
-        </geometry>
-        <material name="grey" />
-    </visual>
-    <collision>
-        <origin xyz="0 0 0" rpy="0 0 0" />
-        <geometry>
-          <sphere radius="0.025" />
-        </geometry>
-    </collision>
-  </link>
-  </link>
+            </geometry>
+        </collision>
+    </link>
+<!--=============================================== GAZEBO ROBOT COLOR ===============================================-->
+    <gazebo reference="base_link">
+        <material>Gazebo/White</material>
+    </gazebo>
+    <gazebo reference="wheel_left_link">
+        <material>Gazebo/Grey</material>
+    </gazebo>
+    <gazebo reference="wheel_right_link">
+        <material>Gazebo/Grey</material>
+    </gazebo>
+    <gazebo reference="caster_front_link">
+        <material>Gazebo/Grey</material>
+        <mu1 value="0.001"/>
+        <mu2 value="0.001"/>
+    </gazebo>
+    <gazebo reference="caster_rear_link">
+        <material>Gazebo/Grey</material>
+        <mu1 value="0.001"/>
+        <mu2 value="0.001"/>
+    </gazebo>
 </robot>
